Commit message: Cartpole experiments

File: assets/urdf/cartpole.urdf (robot description, URDF)
Before this commit: robot cartpole, 3 links, 2 joints
Links:
- link pole: mass 1 -> 5; geometry collision box size=0.2 0.1 1.0; visual box size=0.2 0.1 1.0
Joints:
- joint cart_to_pole: limit effort=1000.0 velocity=8 -> effort=1.0 velocity=9.8
- joint slider_to_cart: limit lower=-4 upper=4 effort=1000.0 velocity=100 -> lower=-8 upper=8 effort=180.0 velocity=1.75
